Commit message: Adição da câmera

File: src/mybot_description/urdf/mybot.xacro (robot description, xacro)
@@ -2,11 +2,12 @@
 <robot name="myrobot"
   xmlns:xacro="http://www.ros.org/wiki/xacro">
+  <!--Arquivo de parametros de montagem do bot-->
   <xacro:include filename="$(find mybot_description)/urdf/mybot.gazebo" />
   <xacro:include filename="$(find mybot_description)/urdf/materials.xacro" />
   <xacro:include filename="$(find mybot_description)/urdf/macros.xacro" />
-  <!--Arquivo de parametros de montagem do bot-->
-<!--
-    Chassis
--->
+  <!--Propriedades da camera-->
+  <xacro:property name="cameraSize" value="0.05"/>
+  <xacro:property name="cameraMass" value="0.1"/>
+  <!--Chassis-->
   <link name='chassis'>
     <pose>0 0 0.1 0 0 0</pose>
@@ -50,7 +51,5 @@
     </visual>
   </link>
-  <!--
-    Roda esquerda
-  -->
+  <!--Roda esquerda-->
   <link name="left_wheel">
     <!--origin xyz="0.1 0.13 0.1" rpy="0 1.5707 1.5707"/-->
@@ -74,7 +73,5 @@
     </inertial>
   </link>
-  <!--
-    Roda direita
-  -->
+  <!--Roda direita-->
   <link name="right_wheel">
     <!--origin xyz="0.1 -0.13 0.1" rpy="0 1.5707 1.5707"/-->
@@ -98,7 +95,5 @@
     </inertial>
   </link>
-  <!--
-    Junta Roda esquerda
-  -->
+  <!--Junta Roda esquerda-->
   <joint type="continuous" name="left_wheel_hinge">
     <origin xyz="0.1 0.15 0" rpy="0 0 0"/>
@@ -109,7 +104,5 @@
     <joint_properties damping="0.0" friction="0.0"/>
   </joint>
-  <!--
-    Junta Roda direita
-  -->
+  <!--Junta Roda direita-->
   <joint type="continuous" name="right_wheel_hinge">
     <origin xyz="0.1 -0.15 0" rpy="0 0 0"/>
@@ -120,5 +113,6 @@
     <joint_properties damping="0.0" friction="0.0"/>
   </joint>
-  <!-- Hokuyo Laser -->
+  <!--Hokuyo Laser-->
+  <!--Junta do Hokuyo Laser-->
   <joint name="hokuyo_joint" type="fixed">
     <axis xyz="0 1 0" />
@@ -127,4 +121,5 @@
     <child link="hokuyo"/>
   </joint>
+<!--Link do Hokuyo Laser-->
   <link name="hokuyo">
     <collision>
@@ -146,3 +141,32 @@
     </inertial>
   </link>
+  <!--Camera-->
+  <!--Junta Camera-->
+  <joint name="camera_joint" type="fixed">
+	  <axis xyz="0 1 0" />
+	  <origin xyz=".2 0 0" rpy="0 0 0"/>
+	  <parent link="chassis"/>
+	  <child link="camera"/>
+  </joint>
+  <!--Link da camera-->
+  <link name="camera">
+	  <collision>
+		  <origin xyz="0 0 0" rpy="0 0 0"/>
+		  <geometry>
+			<box size="${cameraSize} ${cameraSize} ${cameraSize}"/>
+		  </geometry>
+	  </collision>
+	  <visual>
+		  <origin xyz="0 0 0" rpy="0 0 0"/>
+		  <geometry>
+			<box size="${cameraSize} ${cameraSize} ${cameraSize}"/>
+		  </geometry>
+		  <material name="green"/>
+	  </visual>
+	  <inertial>
+		<mass value="${cameraMass}" />
+		<origin xyz="0 0 0" rpy="0 0 0"/>
+		<inertia ixx="1e-6" ixy="0" ixz="0" iyy="1e-6" iyz="0" izz="1e-6" />
+	  </inertial>
+  </link>
 </robot>
